Commit message: roslaunch load.launch works

File: nuturtle_description/urdf/my_turtlebot3.urdf.xacro (robot description, xacro)
@@ -1,6 +1,6 @@
 <?xml version="1.0" ?>
-<robot name="turtlebot3_burger" xmlns:xacro="http://ros.org/wiki/xacro">
-  <xacro:include filename="$(find nuturtle_description)/urdf/common_properties.xacro"/>
-  <xacro:include filename="$(find nuturtle_description)/urdf/turtlebot3_burger.gazebo.xacro"/>
+<robot name="my_turtlebot3" xmlns:xacro="http://ros.org/wiki/xacro">
+  <xacro:include filename="$(find nuturtle_description)/urdf/macro.xacro"/>
+  <!-- <xacro:include filename="$(find nuturtle_description)/urdf/my_turtlebot3.gazebo.xacro"/> -->
   <xacro:property name="diff_params" value="$(find nuturtle_description)/config/diff_params.yaml"/>
   <xacro:property name="dictionary" value="${load_yaml(diff_params)}"/>
@@ -38,5 +38,5 @@
     <parent link="base_link"/>
     <child link="wheel_left_link"/>
-    <origin xyz="0.0 ${wheel_base} 0.023" rpy="-1.57 0 0"/>
+    <origin xyz="0.0 ${wheel_base/2} 0.023" rpy="-1.57 0 0"/>
     <axis xyz="0 0 1"/>
   </joint>
@@ -66,5 +66,5 @@
     <parent link="base_link"/>
     <child link="wheel_right_link"/>
-    <origin xyz="0.0 ${-wheel_base} 0.023" rpy="-1.57 0 0"/>
+    <origin xyz="0.0 ${-wheel_base/2} 0.023" rpy="-1.57 0 0"/>
     <axis xyz="0 0 1"/>
   </joint>

Commit message: Finish task A

File: nuturtle_description/urdf/my_turtlebot3.urdf.xacro (robot description, xacro)
@@ -97,4 +97,11 @@
   </joint>
   <link name="caster_back_link">
+    <visual>
+      <origin rpy="1.57 0 0" xyz="0 0 0"/>
+      <geometry>
+        <box size="0.015 0.005 0.010"/>
+      </geometry>
+      <material name="dark"/>
+    </visual>
     <collision>
       <origin xyz="0 0.001 0" rpy="0 0 0"/>
